File: stm32g030c6t6/stm32g030c6t6.kicad_pcb (KiCad board)
At the start: 2 copper layers, 160 x 55 mm, 73 parts, among them J3 USB_B_Micro, Q1 2N7002, Q2 IRF740, Q3 2N7002, U1 TLP627, U10 XC6206PxxxMR, U2 TLP627, U5 MAX1771xSA

Commit message: Add files via upload
Parts:
- removed the D17 at (-137.0, 43.6)
- removed the D5 at (-153.5, 98.6)
- removed the D6 at (-164.0, 98.6)
- removed the J1 at (-122.3, 92.7)
- removed the R4 at (-29.9, 25.3)
- removed the R6 at (-121.8, 53.3)
- removed the R7 at (-121.8, 59.3)
- removed the R8 at (-145.0, 85.4)
- removed the SW2 at (-121.7, 67.7)
- removed the U1 at (-41.9, 20.2)
- removed the U2 at (-76.1, 43.4)
- added D14: 16CTQ100, Package_TO_SOT_SMD:TO-263-2, F.Cu at (205.9, 126.9)
- added D19: MH-CD42, ИН12А:MH, B.Cu at (198.2, 135.3)
- added D7: К155_ИД1, ИН12А:К155ИД1, F.Cu at (53.2, 126.5)
- added J4: ~, Connector_PinHeader_2.54mm:PinHeader_1x02_P2.54mm_Vertical, B.Cu at (126.3, 127.2)
- added R12: 33kR, Resistor_THT:R_Axial_DIN0309_L9.0mm_D3.2mm_P15.24mm_Horizontal, B.Cu at (88.3, 130.0)
- added R13: 0.05R, Resistor_THT:R_Axial_DIN0309_L9.0mm_D3.2mm_P15.24mm_Horizontal, B.Cu at (57.9, 125.5)
- added R14: 33kR, Resistor_THT:R_Axial_DIN0309_L9.0mm_D3.2mm_P15.24mm_Horizontal, B.Cu at (73.1, 134.5)
- added R5: 510R, Resistor_SMD:R_1206_3216Metric, B.Cu at (172.3, 106.4)
- added SW1: ~, Rotary_Encoder:RotaryEncoder_Alps_EC12E-Switch_Vertical_H20mm, F.Cu at (197.2, 111.2)
- added U3: TLP627, Package_DIP:DIP-4_W7.62mm, B.Cu at (105.1, 126.6)
- added U4: TLP627, Package_DIP:DIP-4_W7.62mm, B.Cu at (105.1, 132.6)
- BT1, BT2, C6, C7, DD1, J5, L1, Y2: moved to B.Cu
- C10: renamed from C17; moved to B.Cu
- C11: renamed from C14; moved to B.Cu
- C12: renamed from C1; moved to B.Cu
- C13: renamed from C3; moved to B.Cu
- C14: renamed from C4; moved to B.Cu
- C15: renamed from C5; moved to B.Cu
- C16: renamed from C10; moved to B.Cu
- C17: renamed from C15; moved to B.Cu
- C18: renamed from C16; moved to B.Cu
- C5: renamed from C2; moved to B.Cu
- C8: renamed from C19; moved to B.Cu
- C9: renamed from C18; moved to B.Cu
- D15: renamed from D7; moved to B.Cu
- D16: value MH-CD42 -> К155_ИД1; footprint Connector_PinHeader_2.54mm:PinHeader_1x06_P2.54mm_Vertical -> ИН12А:К155ИД1; moved to B.Cu
- D17: renamed from D8; moved to B.Cu
- D18: renamed from D14; moved to B.Cu
- J2: footprint Connector_PinHeader_2.54mm:PinHeader_1x02_P2.54mm_Vertical -> Connector_PinSocket_2.54mm:PinSocket_1x03_P2.54mm_Vertical
- J3: renamed from J4; moved to B.Cu
- J6: renamed from J7; moved to B.Cu
- Q3: renamed from Q1; moved to B.Cu
- R10: renamed from R3; moved to B.Cu
- R11: renamed from R5; moved to B.Cu
- R6: renamed from R2; moved to B.Cu
- R7: renamed from R12; moved to B.Cu
- R8: renamed from R11; moved to B.Cu
- R9: renamed from R1; moved to B.Cu
- SW2: renamed from SW1; moved to B.Cu
- moved D13 335.8 mm to (160.7, 109.0)
- moved J5 316.6 mm to (186.5, 135.6), turned to 90 degrees
- moved J6 300.2 mm to (174.7, 135.6), turned to 90 degrees
- moved C9 300.1 mm to (207.2, 114.3)
- moved BT2 299.4 mm to (195.1, 133.4), turned to 135 degrees
- moved DD1 299.0 mm to (185.1, 114.7), turned to -90 degrees
- moved J1 297.7 mm to (213.2, 94.0), turned to 90 degrees
- moved R8 297.1 mm to (202.3, 114.3), turned to 180 degrees
- moved J2 293.7 mm to (195.5, 123.7)
- moved C8 289.3 mm to (207.2, 116.7)
- moved Y1 285.3 mm to (178.7, 107.3), turned to 90 degrees
- moved C10 284.1 mm to (193.2, 108.1), turned to 90 degrees
- moved SW2 283.9 mm to (183.4, 100.8)
- moved Y2 280.8 mm to (186.0, 92.1), turned to 180 degrees
- moved BT1 280.3 mm to (204.1, 100.7)
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- renumbered C12 to C1, C13 to C2, C11 to C3, C21 to C4, D15 to D1, D11 to D10, D4 to D11, D2 to D12, D19 to D13, D13 to D2, D10 to D3, D12 to D4, D18 to D5, D9 to D6, D3 to D8, D1 to D9, J3 to J1, Q2 to Q1, Q3 to Q2, R14 to R1, R10 to R2, R13 to R3, R9 to R4, U5 to U1, U10 to U2
Connections:
- D11 pad 1: Net-(J2-Pad2) -> Net-(D1-Pad1)
- D11 pad 10: Net-(D6-Pad8) -> Net-(D2-Pad10)
- D11 pad 11: Net-(D6-Pad2) -> Net-(D6-Pad8)
- D11 pad 2: Net-(D6-Pad1) -> Net-(D6-Pad9)
- D11 pad 3: Net-(D6-Pad9) -> Net-(D4-Pad3)
- D11 pad 4: Net-(D6-Pad11) -> Net-(D2-Pad4)
- D11 pad 5: Net-(D6-Pad14) -> Net-(D2-Pad5)
- D11 pad 6: Net-(D6-Pad16) -> Net-(D6-Pad1)
- D11 pad 7: Net-(D6-Pad15) -> Net-(D6-Pad2)
- D11 pad 8: Net-(D6-Pad13) -> Net-(D2-Pad8)
- D11 pad 9: Net-(D6-Pad10) -> Net-(D2-Pad9)
- D12 pad 1: Net-(J2-Pad1) -> Net-(D3-Pad1)
- D12 pad 10: Net-(D6-Pad8) -> Net-(D2-Pad10)
- D12 pad 11: Net-(D6-Pad2) -> Net-(D6-Pad8)
- D12 pad 2: Net-(D6-Pad1) -> Net-(D6-Pad9)
- D12 pad 3: Net-(D6-Pad9) -> Net-(D4-Pad3)
- D12 pad 4: Net-(D6-Pad11) -> Net-(D2-Pad4)
- D12 pad 5: Net-(D6-Pad14) -> Net-(D2-Pad5)
- D12 pad 6: Net-(D6-Pad16) -> Net-(D6-Pad1)
- D12 pad 7: Net-(D6-Pad15) -> Net-(D6-Pad2)
- D12 pad 8: Net-(D6-Pad13) -> Net-(D2-Pad8)
- D12 pad 9: Net-(D6-Pad10) -> Net-(D2-Pad9)
- D16 pad 1: /5V_BAT -> Net-(D6-Pad1)
- D16 pad 2: GNDD -> Net-(D6-Pad2)
- D16 pad 3: Net-(BT2-Pad1) -> /D1_X4
- D16 pad 4: Net-(BT2-Pad2) -> /D1_X3
- D16 pad 5: GNDD -> +5V
- D16 pad 6: /5V_USB -> /D1_X2
- D5 pad 4: /LED_FRONT_PWM -> /PWM_WS2812B
- D8 pad 1: Net-(J2-Pad2) -> Net-(D3-Pad1)
- D9 pad 1: Net-(J2-Pad1) -> Net-(D1-Pad1)
- DD1 pad 13: /D2_X1 -> unconnected-(DD1-Pad13)
- DD1 pad 14: /D2_X2 -> unconnected-(DD1-Pad14)
- DD1 pad 15: /D2_X3 -> unconnected-(DD1-Pad15)
- DD1 pad 16: /D2_X4 -> unconnected-(DD1-Pad16)
- DD1 pad 37: /D1_X1 -> /D2_X1
- DD1 pad 38: /D1_X2 -> /D2_X2
- DD1 pad 39: /D1_X3 -> /D2_X3
- DD1 pad 40: /D1_X4 -> /D2_X4
- DD1 pad 41: unconnected-(DD1-Pad41) -> /D1_X1
- DD1 pad 42: unconnected-(DD1-Pad42) -> /D1_X2
- DD1 pad 43: unconnected-(DD1-Pad43) -> /D1_X3
- DD1 pad 44: unconnected-(DD1-Pad44) -> /D1_X4
- DD1 pad 7: /GND -> GNDD
- J2 pad 1: Net-(J2-Pad1) -> GNDD
- J2 pad 2: Net-(J2-Pad2) -> /ADC_IN2
- R6 pad 1: /LED_PWM -> /LED_FRONT_PWM
- R7 pad 2: /CLK_Encoder -> /DT_Encoder
- R8 pad 2: /DT_Encoder -> /CLK_Encoder
Routing:
- net /D2_X1: track 0.00 -> 152.4 mm
- net /D2_X2: track 0.00 -> 148.9 mm
- net +3.3V: track 0.00 -> 147.1 mm, vias 0 -> 3
- net /D2_X3: track 0.00 -> 143.0 mm
- net /D2_X4: track 0.00 -> 139.4 mm
- net GNDD: track 0.00 -> 109.2 mm, vias 0 -> 18
- net /LP2: track 0.00 -> 97.1 mm, vias 0 -> 1
- net /LP1: track 0.00 -> 93.3 mm, vias 0 -> 1
- net /LED_FRONT_PWM: track 0.00 -> 82.4 mm
- net /HVT: track 0.00 -> 78.9 mm, vias 0 -> 1
- net /PWM_WS2812B: track 0.00 -> 68.0 mm, vias 0 -> 3
- net Net-(D1-Pad1): track 0.00 -> 62.9 mm, vias 0 -> 2
- net Net-(D3-Pad1): track 0.00 -> 60.0 mm, vias 0 -> 2
- net /5V_USB: track 0.00 -> 54.2 mm
- net Net-(D6-Pad8): track 0.00 -> 47.6 mm
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- added copper zone on F.Cu, net +5V
- added copper zone on B.Cu, net GNDD
Other:
- board size 160 x 55 mm -> 170.9 x 50 mm
- board text added: "RV1"
- board text added: "~"

Commit message: Add files via upload
Parts:
- added J6: ~, Connector_PinHeader_2.54mm:PinHeader_1x02_P2.54mm_Vertical, F.Cu at (227.5, 62.1)
- moved C11 79.1 mm to (195.3, 60.8)
- moved D17 79.1 mm to (245.1, 58.2)
- moved D8 79.1 mm to (192.8, 57.0)
- moved C10 79.1 mm to (205.5, 60.9)
- moved C12 79.1 mm to (117.0, 56.7)
- moved C13 79.1 mm to (192.4, 60.8)
- moved C2 79.1 mm to (214.7, 36.5)
- moved C6 79.1 mm to (226.9, 26.7)
- moved C7 79.1 mm to (223.7, 26.7)
- moved D14 79.1 mm to (123.7, 57.7)
- moved D15 79.1 mm to (110.8, 24.5)
- moved D3 79.1 mm to (110.8, 40.0)
- moved J1 79.1 mm to (234.7, 55.0)
- moved J5 79.1 mm to (225.7, 66.9)
- moved L1 79.1 mm to (90.1, 59.3)
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- renumbered C12 to C1, C16 to C10, C3 to C11, C1 to C12, C2 to C13, C11 to C14, C17 to C15, C18 to C16, C10 to C17, C9 to C18, C8 to C19, C5 to C2, C4 to C21, C13 to C3, C14 to C4, C15 to C5, D9 to D1, D3 to D10, D10 to D11, D4 to D12, D2 to D13, D18 to D14, D1 to D15, D19 to D16, D14 to D17, D5 to D18, D13 to D19, D12 to D2, D8 to D3, D11 to D4, D7 to D5, D16 to D6, D15 to D7, D17 to D8, D6 to D9, J2 to J1, J4 to J2, J1 to J3, J3 to J4, J6 to J7, Q3 to Q1, Q1 to Q2, Q2 to Q3, R9 to R1, R2 to R10, R8 to R11, R7 to R12, R3 to R13, R1 to R14, R6 to R2, R10 to R3, R5 to R4, R11 to R5, R13 to R6, R12 to R7, R14 to R8, R4 to R9, SW2 to SW1, SW1 to SW2, U4 to U1, U2 to U10, U3 to U2, U1 to U5
Routing:
- net /PWM_WS2812B: track 68.0 -> 66.5 mm
- net (no net): vias 0 -> 4
Other:
- outline, holes or cut-outs redrawn
