File: stm32g030c6t6/stm32g030c6t6.kicad_sch (KiCad schematic)
At the start: 73 parts, among them J3 USB_B_Micro, Q1 2N7002, Q2 IRF740, Q3 2N7002, U1 TLP627, U10 XC6206PxxxMR, U2 TLP627, U5 MAX1771xSA

Commit message: Add files via upload
Connections:
- net at D1.11, D3.11: now also D5.15 (V1); no longer D5.2 (V9)
- net at D1.2, D3.2: now also D5.16 (V0); no longer D5.1 (V8)
- net at D1.3, D3.3: now also D5.2 (V9); no longer D5.9 (V3)
- net at D1.4, D3.4: now also D5.1 (V8); no longer D5.11 (V6)
- net at D1.5, D3.5: now also D5.10 (V7); no longer D5.14 (V5)
- net at D1.6, D3.6: now also D5.11 (V6); no longer D5.16 (V0)
- net at D1.7, D3.7: now also D5.14 (V5); no longer D5.15 (V1)
- net at D1.9, D3.9: now also D5.9 (V3); no longer D5.10 (V7)
Other:
- moved on the sheet: D5

Commit message: Add files via upload
Parts:
- added J6: ~, Connector_PinHeader_2.54mm:PinHeader_1x02_P2.54mm_Vertical, symbol Connector:Conn_01x02_Female
- D16: footprint Connector_PinHeader_2.54mm:PinHeader_1x06_P2.54mm_Vertical -> ИН12А:MH
- R6, R7, R8: footprint Resistor_THT:R_Axial_DIN0414_L11.9mm_D4.5mm_P20.32mm_Horizontal -> Resistor_THT:R_Axial_DIN0309_L9.0mm_D3.2mm_P15.24mm_Horizontal
Connections:
- net GND is gone; now on net GNDD: DD1.7 (VSS/VSSA)
- net LED_PWM is gone; now on net LED_FRONT_PWM: R2.1
- net PC13 is gone; now on net LED_C13: R4.2
- net +5V: now also J6.1 (Pin_1)
- net 5V_BAT: now also D17.1 (A); no longer D17.3 (A)
- net 5V_USB: now also D17.3 (A); no longer D17.1 (A)
- net CLK_Encoder: now also R11.2, SW2.A; no longer R12.2, SW2.B
- net D1_X1: now also D6.7 (X3), DD1.41 (PD3); no longer D6.3 (X1), DD1.37 (PA15)
- net D1_X2: now also DD1.42 (PB3); no longer DD1.38 (PD0)
- net D1_X3: now also D6.4 (X4), DD1.43 (PB4); no longer D6.7 (X3), DD1.39 (PD1)
- net D1_X4: now also D6.3 (X1), DD1.44 (PB5); no longer D6.4 (X4), DD1.40 (PD2)
- net D2_X1: now also DD1.37 (PA15); no longer DD1.13 (PA2)
- net D2_X2: now also D5.4 (X4), DD1.38 (PD0); no longer D5.6 (X2), DD1.14 (PA3)
- net D2_X3: now also D5.6 (X2), DD1.39 (PD1); no longer D5.7 (X3), DD1.15 (PA4)
- net D2_X4: now also D5.7 (X3), DD1.40 (PD2); no longer D5.4 (X4), DD1.16 (PA5)
- net DT_Encoder: now also R12.2, SW2.B; no longer R11.2, SW2.A
- net GNDD: now also J6.2 (Pin_2)
- net LED_FRONT_PWM: no longer D18.4 (DIN)
- net PWM_WS2812B: now also D18.4 (DIN)
- net at D1.1 (Анод), J2.1 (Pin_1): now also D4.1 (Анод); no longer D2.1 (Анод)
- net at D2.10, D4.10: now also D6.10 (V7); no longer D6.8 (V2)
- net at D2.11, D4.11: now also D6.8 (V2); no longer D6.2 (V9)
- net at D2.2, D4.2: now also D6.9 (V3); no longer D6.1 (V8)
- net at D2.3, D4.3: now also D6.11 (V6); no longer D6.9 (V3)
- net at D2.4, D4.4: now also D6.14 (V5); no longer D6.11 (V6)
- net at D2.5, D4.5: now also D6.16 (V0); no longer D6.14 (V5)
- net at D2.6, D4.6: now also D6.1 (V8); no longer D6.16 (V0)
- net at D2.7, D4.7: now also D6.2 (V9); no longer D6.15 (V1)
- net at D2.8, D4.8: now also D6.15 (V1); no longer D6.13 (V4)
- net at D2.9, D4.9: now also D6.13 (V4); no longer D6.10 (V7)
- net at D3.1 (Анод), J2.2 (Pin_2): now also D2.1 (Анод); no longer D4.1 (Анод)
- net at D1.10, D3.10: now also D5.10 (V7); no longer D5.8 (V2)
- net at D1.11, D3.11: now also D5.8 (V2); no longer D5.15 (V1)
- net at D1.2, D3.2: now also D5.9 (V3); no longer D5.16 (V0)
- net at D1.3, D3.3: now also D5.11 (V6); no longer D5.2 (V9)
- net at D1.4, D3.4: now also D5.14 (V5); no longer D5.1 (V8)
- net at D1.5, D3.5: now also D5.16 (V0); no longer D5.10 (V7)
- net at D1.6, D3.6: now also D5.1 (V8); no longer D5.11 (V6)
- net at D1.7, D3.7: now also D5.2 (V9); no longer D5.14 (V5)
- net at D1.8, D3.8: now also D5.15 (V1); no longer D5.13 (V4)
- net at D1.9, D3.9: now also D5.13 (V4); no longer D5.9 (V3)
Other:
- moved on the sheet: D5, J2
